File: hardware/v3.9/BusPirate-v3.9-SSOP.sch (EAGLE design)
At the start: 40 parts, among them CON1 CON_JST_PH_10, CON2 CON_JST_PH_6, CON3 CON-USB-F-MICRO-B, IC1 PIC24FJ64GA002, IC3 4066, IC4 IC_FT230X-SSOP-16

Commit message: - Change IO connector to 0.1 PTH right angled shrouded - Change USB connector - Change LEDs from 0603 to 0804 - Fix texts orientation
Parts:
- removed R5: 10K, dp_devices:RESISTORR603
- added RN4: 10k, dp_devices:RNETWORK
- CON1: value CON_JST_PH_10 -> CON_HEADER_1X10-RIGHT_ANGLED_PTH_SHROUDED; device dp_devices.v6:CON_JST_PH_10 -> dp_devices.v6:CON_HEADER_1X10-RIGHT_ANGLED_PTH_SHROUDED
- CON2: value CON_JST_PH_6 -> CON_HEADER_1X06-PTH; device dp_devices.v6:CON_JST_PH_6 -> dp_devices.v6:CON_HEADER_1X06-PTH
- LED1, LED1A, LED2, LED2A, LED3, LED3A, LED4, LED4A: device dp_devices:LED-0603 -> dp_devices.v6:LED-0805
Connections:
- removed net N$1: IC3A.B, RN3D.1
- removed net N$2: IC3C.B, RN3C.1
- removed net N$4: IC3D.B, RN3B.1
- removed net N$5: IC3B.B, RN3A.1
- removed net TP0: IC1.RA2/CN30/OSCI/CLKI
- new net N$10: IC3A.A, IC3B.A, IC3C.A, RN3A.1, RN3B.1, RN3C.1, RN3D.1, RN4A.2
- new net TP1: IC1.RB2/AN4/RP2/CN6/C1IN-/SDA2
- new net V33PU: IC1.RB3/AN5/RP3/CN7/C1IN+/SCL2, IC3B.C, RN4C.1
- new net V50PU: IC1.RA2/CN30/OSCI/CLKI, IC3C.C, RN4D.1
- net $N26: now also CON3CON1.VUSB; no longer CON3USB.VUSB
- net +3V3: now also CON2.2; no longer CON2CON.2
- net ADC: now also CON1.5; no longer CON1CON.6
- net AUX1: now also CON1.6, RN4A.1; no longer CON1CON.5
- net CLK: now also CON1.9, RN3D.2; no longer CON1CON.2, RN3A.2
- net CS: now also CON1.7, RN3B.2; no longer CON1CON.4, RN3C.2
- net GND: now also CON1.1, CON2.3, CON3CON1.GND, CON3GPINS.P$1, CON3GPINS.P$2, CON3GPINS.P$3, CON3GPINS.P$4, CON3GPINS.P$5, CON3GPINS.P$6, RN4B.2, RN4C.2, RN4D.2; no longer CON1CON.10, CON1CON_GND.1, CON1CON_GND.2, CON2CON.3, CON2CON_GND.1, CON2CON_GND.2, CON3BODY.BODY@1, CON3BODY.BODY@2, CON3BODY.BODY@3, CON3BODY.BODY@4, CON3USB.GND, IC1.RB2/AN4/RP2/CN6/C1IN-/SDA2, IC1.RB3/AN5/RP3/CN7/C1IN+/SCL2
- net MCLR: now also CON2.1; no longer CON2CON.1
- net MISO: now also CON1.8, RN3C.2; no longer CON1CON.3, RN3B.2
- net MOSI: now also CON1.10, RN3A.2; no longer CON1CON.1, RN3D.2
- net N$15: now also CON3CON1.D+; no longer CON3USB.D+
- net N$16: now also CON3CON1.D-; no longer CON3USB.D-
- net PGC: now also CON2.5; no longer CON2CON.5
- net PGD: now also CON2.4; no longer CON2CON.4
- net PULLUPEN: now also RN4B.1; no longer IC3B.C, IC3C.C, IC3D.C, R5.2
- net SWV33: now also CON1.3, IC3B.B; no longer CON1CON.8
- net SWV50: now also CON1.2, IC3C.B; no longer CON1CON.9
- net VEXTERN: now also CON1.4, IC3A.B; no longer CON1CON.7, IC3A.A, IC3B.A, IC3C.A, IC3D.A
- net VUSB: no longer R5.1
Other:
- note added: "Bus Pirate v3.9"
- note added: "Ea"
- note added: "Eb"
- note added: "Ec"
- note added: "Ian Lesnet 2018"
- note added: "Ya"
- note added: "Yb"
- note added: "Yc"
- note added: "Za"
- note added: "Zb"
- note added: "Zc"
- note removed: "Bus Pirate v3.8a"
- note removed: "Ian Lesnet 2014"
- moved on the sheet: C3, IC3A, IC3B, IC3C, IC3P, RN3A, RN3B, RN3C, RN3D
